File: ADC_modul.sch (KiCad schematic (older format))
At the start: 101 parts

Commit message: Add files via upload
Parts:
- removed C? (x19): 100n, symbol C_Small
- removed L? (x4): 910nH, symbol L
- removed P?: CONN_01X04, symbol CONN_01X04
- removed R? (x8): 220, symbol R
- added C? (x4): 4.7u, symbol C_Small
- added C? (x2): 10u, symbol C_Small
- added C? (x9): 100n, symbol C_Small
- added C?: 0.1u, symbol C_Small
- added C?: 1u, symbol C_Small
- added C?: 22u, symbol CP
- added C?: 1u, symbol CP
- added L? (x4): 820n, symbol L_Core_Ferrite_Small
- added L?: 100u, symbol L_Core_Ferrite_Small
- added P?: ext_clk_enable, symbol CONN_01X03
- added P?: diff_ext_clock, symbol CONN_01X03
- added P?: ext_clk, symbol CONN_01X04
- added P?: A, symbol CONN_01X32
- added P?: B, symbol CONN_01X32
- added P?: C, symbol CONN_01X32
- added P?: D, symbol CONN_01X32
- added P?: CONN_01X06, symbol CONN_01X06
- added R? (x4): 50, symbol R
- added R? (x12): 33, symbol R
- added R? (x2): 10k, symbol R
- added R? (x63): 22, symbol R_Small
- added R? (x8): DNI, symbol R_Small
- added R? (x2): 4.7k, symbol R
- added R?: 30k, symbol R
- added R?: 24k, symbol R
- added U?: SN74LVC2G07, MODULE, symbol SN74LVC2G07
- added U?: BD00HC0WEFJ, MODULE, symbol BD00HC0WEFJ
- L? (x2): value L_Core_Ferrite_Small -> 100u
- T? (x4): value ADT4-6WT -> ADT1-1WT
Connections:
- net labels added: D0(16bit), D0B, D1(16bit), D1B, D2B, D3B, D4B, D5B, D6B, D7B, D8B, D9B, GND, GNDPWR, VDDA, cs1, cs2, sclk, sdi, sdo
- wire segments 154 -> 346
Other:
- moved on the sheet: C?, L?, P?, R?, T?, U?, v?
